File: ponderadaPcb/ponderadaPcb.kicad_pcb (KiCad board)
At the start: 2 copper layers, 4 parts, among them Q1 BF457, U1 Pico

Commit message: update esquematico
Routing:
- net Net-(D1-K): track 13.0 -> 15.8 mm
